File: Hardware/KiCad/Mcc18.kicad_pcb (KiCad board)
At the start: 2 copper layers, 47 parts, among them Q1 IRFP4321PbF, U1 LTSP_25-NP, U2 DRIVER_(INEP), U3 LM7812_TO220, U4 Signals_MCC, U5 ZCS

Commit message: initial commit
Parts:
- D1, Q1: footprint Package_TO_SOT_THT:TO-247-3_Horizontal_TabUp -> MCCplaca:TO-247-3_Horizontal_TabUp
- L1: footprint MCC:NEE-42-20-DE -> MCCplaca:NEE-42-20-DE
- U1: footprint MCC:LTSP_25-NP -> MCCplaca:LTSP_25-NP
- U2: footprint MCC:Driver_(INEP) -> MCCplaca:Driver_(INEP)
- U4: footprint MCC:Signals -> MCCplaca:Signals
- U5: footprint MCC:ZCS18 -> MCCplaca:ZCS18
- moved C7 6.54 mm to (139.0, 29.1), turned to 180 degrees
- moved C6 4.38 mm to (139.0, 31.2), turned to 180 degrees
- moved L2 3.70 mm to (142.0, 30.3), turned to 90 degrees
- moved U4 2.29 mm to (152.9, 80.3)
- moved U5 0.63 mm to (85.3, 115.6)
Connections:
- net +18V_OUT renamed /+18V_OUT
- net B+ renamed /+B
- net B- renamed /-B
- net BatOVInterrupt renamed /BatOVInterrupt
- net Gate renamed /Gate
- net Ipanel renamed /Ipanel_adc+
- net Ipanel_Ref renamed GND
- net Ipanel_SIG renamed /Ipanel+
- net PWM renamed /PWM
- net Source renamed /Source
- net Vbat renamed /Vbat_adc+
- net Vp+ renamed /+Vp
- net Vp- renamed /-Vp
- net Vpanel renamed /Vpanel_adc+
- C6 pad 1: Net-(C6-Pad1) -> +5VA
- C7 pad 1: +5VA -> +5V
- L2 pad 1: Net-(C6-Pad1) -> +5VA
- L2 pad 2: +5VA -> +5V
- U4 pad 17: Net-(C6-Pad1) -> +5VA
Routing:
- net /-Vp: track 145.3 -> 347.1 mm, vias 0 -> 3
- net /+Vp: track 108.1 -> 307.6 mm, vias 2 -> 5
- net /+B: track 141.8 -> 336.5 mm, vias 0 -> 3
- net /-B: track 86.2 -> 273.7 mm, vias 0 -> 3
- net GNDA: track 37.4 -> 140.2 mm, vias 1 -> 14
- net GND: track 225.3 -> 301.6 mm, vias 6 -> 5
- net +5V: track 118.6 -> 128.7 mm, vias 2 -> 3
- net /Vpanel_adc+: track 49.2 -> 54.9 mm
- net Net-(C6-Pad1): track 4.58 -> 0.00 mm
- net /+18V_OUT: track 71.2 -> 75.7 mm
- net /Ipanel_adc+: track 36.0 -> 40.3 mm
- net /Ipanel+: track 81.3 -> 84.9 mm
- net +5VA: track 2.14 -> 5.45 mm
- net /PWM: track 119.2 -> 116.2 mm, vias 4 -> 3
- net Net-(U1-Pad3): track 17.2 -> 16.2 mm
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- added copper zone on B.Cu, net /+B
- added copper zone on B.Cu, net /+Vp
- added copper zone on B.Cu, net /-B
- added copper zone on F.Cu, net /Source
- added copper zone on B.Cu, net GND
