File: Hardware/Hall sensor/Cuk converter/KiCad/Mcc18.kicad_pcb (KiCad board)
At the start: 2 copper layers, 202.2 x 107.2 mm, 47 parts, among them Q1 IRFP4321PbF, U1 LTSP_25-NP, U2 DRIVER_(INEP), U3 LM7812_TO220, U4 Signals_MCC, U5 ZCS

Commit message: created signals PCB
Routing:
- net /+B: track 292.6 -> 291.9 mm
Changed lines of the file:
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@@
     (thickness 1.6)
     (drawings 9)
-    (tracks 511)
+    (tracks 509)
     (zones 0)
     (modules 47)
@@
     (add_net "Net-(U1-Pad3)")
   )
+  (module MCCplaca:Signals (layer B.Cu)
+    (at 152.908 80.264 90)
+    (fp_text reference U4 (at 0 -0.5 90) (layer B.SilkS)
+      (effects (font (size 1 1) (thickness 0.15)) (justify mirror))
+    )
+    (fp_text value Signals_MCC (at 0 0.5 90) (layer B.Fab)
+      (effects (font (size 1 1) (thickness 0.15)) (justify mirror))
+    )
+    (fp_line (start 46.99 -11.43) (end 36.83 -11.43) (layer B.SilkS) (width 0.15))
+    (fp_line (start 46.99 -13.97) (end 46.99 -11.43) (layer B.SilkS) (width 0.15))
+    (fp_line (start 36.83 -13.97) (end 46.99 -13.97) (layer B.SilkS) (width 0.15))
+    (fp_line (start 36.83 -11.43) (end 36.83 -13.97) (layer B.SilkS) (width 0.15))
+    (fp_line (start 35.56 -11.43) (end 25.4 -11.43) (layer B.SilkS) (width 0.15))
+    (fp_line (start 35.56 -13.97) (end 35.56 -11.43) (layer B.SilkS) (width 0.15))
+    (fp_line (start 25.4 -13.97) (end 35.56 -13.97) (layer B.SilkS) (width 0.15))
+    (fp_line (start 25.4 -11.43) (end 25.4 -13.97) (layer B.SilkS) (width 0.15))
+    (fp_line (start 25.654 -11.43) (end 25.4 -11.43) (layer B.SilkS) (width 0.15))
+    (fp_line (start 0 -11.43) (end 10.16 -11.43) (layer B.SilkS) (width 0.15))
+    (fp_line (start 0 -13.97) (end 0 -11.43) (layer B.SilkS) (width 0.15))
+    (fp_line (start 10.16 -13.97) (end 0 -13.97) (layer B.SilkS) (width 0.15))
+    (fp_line (start 10.16 -11.43) (end 10.16 -13.97) (layer B.SilkS) (width 0.15))
+    (fp_line (start 24.13 -11.43) (end 11.43 -11.43) (layer B.SilkS) (width 0.15))
+    (fp_line (start 24.13 -11.684) (end 24.13 -11.43) (layer B.SilkS) (width 0.15))
+    (fp_line (start 24.13 -13.97) (end 24.13 -11.684) (layer B.SilkS) (width 0.15))
+    (fp_line (start 11.43 -13.97) (end 24.13 -13.97) (layer B.SilkS) (width 0.15))
+    (fp_line (start 11.43 -11.43) (end 11.43 -13.97) (layer B.SilkS) (width 0.15))
+    (pad 17 thru_hole circle (at 45.72 -12.7 90) (size 1.524 1.524) (drill 0.762) (layers *.Cu *.Mask)
+      (net 28 +5VA))
+    (pad 1 thru_hole circle (at 1.27 -12.7 90) (size 1.524 1.524) (drill 0.762) (layers *.Cu *.Mask)
+      (net 50 /-Vp))
+    (pad 2 thru_hole circle (at 3.81 -12.7 90) (size 1.524 1.524) (drill 0.762) (layers *.Cu *.Mask)
+      (net 37 /+Vp))
+    (pad 3 thru_hole circle (at 6.35 -12.7 90) (size 1.524 1.524) (drill 0.762) (layers *.Cu *.Mask)
+      (net 27 GNDA))
+    (pad 4 thru_hole circle (at 8.89 -12.7 90) (size 1.524 1.524) (drill 0.762) (layers *.Cu *.Mask)
+      (net 44 /Vpanel_adc+))
+    (pad 5 thru_hole circle (at 12.7 -12.7 90) (size 1.524 1.524) (drill 0.762) (layers *.Cu *.Mask)
+      (net 27 GNDA))
+    (pad 6 thru_hole circle (at 15.24 -12.7 90) (size 1.524 1.524) (drill 0.762) (layers *.Cu *.Mask)
+      (net 49 /Ipanel+))
+    (pad 7 thru_hole circle (at 17.78 -12.7 90) (size 1.524 1.524) (drill 0.762) (layers *.Cu *.Mask)
+      (net 41 GND))
+    (pad 8 thru_hole circle (at 20.32 -12.7 90) (size 1.524 1.524) (drill 0.762) (layers *.Cu *.Mask)
+      (net 27 GNDA))
+    (pad 9 thru_hole circle (at 22.86 -12.7 90) (size 1.524 1.524) (drill 0.762) (layers *.Cu *.Mask)
+      (net 45 /Ipanel_adc+))
+    (pad 10 thru_hole circle (at 26.67 -12.7 90) (size 1.524 1.524) (drill 0.762) (layers *.Cu *.Mask)
+      (net 48 /+B))
+    (pad 11 thru_hole circle (at 29.21 -12.7 90) (size 1.524 1.524) (drill 0.762) (layers *.Cu *.Mask)
+      (net 38 /-B))
+    (pad 12 thru_hole circle (at 31.75 -12.7 90) (size 1.524 1.524) (drill 0.762) (layers *.Cu *.Mask)
+      (net 27 GNDA))
+    (pad 13 thru_hole circle (at 34.29 -12.7 90) (size 1.524 1.524) (drill 0.762) (layers *.Cu *.Mask)
+      (net 43 /Vbat_adc+))
+    (pad 14 thru_hole circle (at 38.1 -12.7 90) (size 1.524 1.524) (drill 0.762) (layers *.Cu *.Mask)
+      (net 47 /BatOVInterrupt))
+    (pad 15 thru_hole circle (at 40.64 -12.7 90) (size 1.524 1.524) (drill 0.762) (layers *.Cu *.Mask)
+      (net 46 /PWM))
+    (pad 16 thru_hole circle (at 43.18 -12.7 90) (size 1.524 1.524) (drill 0.762) (layers *.Cu *.Mask)
+      (net 27 GNDA))
+    (model "C:/GitZenite/MCC18/Hardware/Shunt sensor/MCC_bibliotecas/MCCplaca.pretty/3D/SignalPCB.stp"
+      (offset (xyz -28.44799957275391 -33.01999950408936 6.984999895095826))
+      (scale (xyz 1 1 1))
+      (rotate (xyz 180 0 0))
+    )
+  )
   (module MCCplaca:hs10425 (layer B.Cu)
     (at 194.31 110.49)
@@
       (rotate (xyz -90 0 0))
     )
-  )
-  (module MCCplaca:Signals (layer B.Cu)
-    (at 152.908 80.264 90)
-    (fp_text reference U4 (at 0 -0.5 90) (layer B.SilkS)
-      (effects (font (size 1 1) (thickness 0.15)) (justify mirror))
-    )
-    (fp_text value Signals_MCC (at 0 0.5 90) (layer B.Fab)
-      (effects (font (size 1 1) (thickness 0.15)) (justify mirror))
-    )
-    (fp_line (start 11.43 -11.43) (end 11.43 -13.97) (layer B.SilkS) (width 0.15))
-    (fp_line (start 11.43 -13.97) (end 24.13 -13.97) (layer B.SilkS) (width 0.15))
-    (fp_line (start 24.13 -13.97) (end 24.13 -11.684) (layer B.SilkS) (width 0.15))
-    (fp_line (start 24.13 -11.684) (end 24.13 -11.43) (layer B.SilkS) (width 0.15))
-    (fp_line (start 24.13 -11.43) (end 11.43 -11.43) (layer B.SilkS) (width 0.15))
-    (fp_line (start 10.16 -11.43) (end 10.16 -13.97) (layer B.SilkS) (width 0.15))
-    (fp_line (start 10.16 -13.97) (end 0 -13.97) (layer B.SilkS) (width 0.15))
-    (fp_line (start 0 -13.97) (end 0 -11.43) (layer B.SilkS) (width 0.15))
-    (fp_line (start 0 -11.43) (end 10.16 -11.43) (layer B.SilkS) (width 0.15))
-    (fp_line (start 25.654 -11.43) (end 25.4 -11.43) (layer B.SilkS) (width 0.15))
-    (fp_line (start 25.4 -11.43) (end 25.4 -13.97) (layer B.SilkS) (width 0.15))
-    (fp_line (start 25.4 -13.97) (end 35.56 -13.97) (layer B.SilkS) (width 0.15))
-    (fp_line (start 35.56 -13.97) (end 35.56 -11.43) (layer B.SilkS) (width 0.15))
-    (fp_line (start 35.56 -11.43) (end 25.4 -11.43) (layer B.SilkS) (width 0.15))
-    (fp_line (start 36.83 -11.43) (end 36.83 -13.97) (layer B.SilkS) (width 0.15))
-    (fp_line (start 36.83 -13.97) (end 46.99 -13.97) (layer B.SilkS) (width 0.15))
-    (fp_line (start 46.99 -13.97) (end 46.99 -11.43) (layer B.SilkS) (width 0.15))
-    (fp_line (start 46.99 -11.43) (end 36.83 -11.43) (layer B.SilkS) (width 0.15))
-    (pad 16 thru_hole circle (at 43.18 -12.7 90) (size 1.524 1.524) (drill 0.762) (layers *.Cu *.Mask)
-      (net 27 GNDA))
-    (pad 15 thru_hole circle (at 40.64 -12.7 90) (size 1.524 1.524) (drill 0.762) (layers *.Cu *.Mask)
-      (net 46 /PWM))
-    (pad 14 thru_hole circle (at 38.1 -12.7 90) (size 1.524 1.524) (drill 0.762) (layers *.Cu *.Mask)
-      (net 47 /BatOVInterrupt))
-    (pad 13 thru_hole circle (at 34.29 -12.7 90) (size 1.524 1.524) (drill 0.762) (layers *.Cu *.Mask)
-      (net 43 /Vbat_adc+))
-    (pad 12 thru_hole circle (at 31.75 -12.7 90) (size 1.524 1.524) (drill 0.762) (layers *.Cu *.Mask)
-      (net 27 GNDA))
-    (pad 11 thru_hole circle (at 29.21 -12.7 90) (size 1.524 1.524) (drill 0.762) (layers *.Cu *.Mask)
-      (net 38 /-B))
-    (pad 10 thru_hole circle (at 26.67 -12.7 90) (size 1.524 1.524) (drill 0.762) (layers *.Cu *.Mask)
-      (net 48 /+B))
-    (pad 9 thru_hole circle (at 22.86 -12.7 90) (size 1.524 1.524) (drill 0.762) (layers *.Cu *.Mask)
-      (net 45 /Ipanel_adc+))
-    (pad 8 thru_hole circle (at 20.32 -12.7 90) (size 1.524 1.524) (drill 0.762) (layers *.Cu *.Mask)
-      (net 27 GNDA))
-    (pad 7 thru_hole circle (at 17.78 -12.7 90) (size 1.524 1.524) (drill 0.762) (layers *.Cu *.Mask)
-      (net 41 GND))
-    (pad 6 thru_hole circle (at 15.24 -12.7 90) (size 1.524 1.524) (drill 0.762) (layers *.Cu *.Mask)
-      (net 49 /Ipanel+))
-    (pad 5 thru_hole circle (at 12.7 -12.7 90) (size 1.524 1.524) (drill 0.762) (layers *.Cu *.Mask)
-      (net 27 GNDA))
-    (pad 4 thru_hole circle (at 8.89 -12.7 90) (size 1.524 1.524) (drill 0.762) (layers *.Cu *.Mask)
-      (net 44 /Vpanel_adc+))
-    (pad 3 thru_hole circle (at 6.35 -12.7 90) (size 1.524 1.524) (drill 0.762) (layers *.Cu *.Mask)
-      (net 27 GNDA))
-    (pad 2 thru_hole circle (at 3.81 -12.7 90) (size 1.524 1.524) (drill 0.762) (layers *.Cu *.Mask)
-      (net 37 /+Vp))
-    (pad 1 thru_hole circle (at 1.27 -12.7 90) (size 1.524 1.524) (drill 0.762) (layers *.Cu *.Mask)
-      (net 50 /-Vp))
-    (pad 17 thru_hole circle (at 45.72 -12.7 90) (size 1.524 1.524) (drill 0.762) (layers *.Cu *.Mask)
-      (net 28 +5VA))
   )
   (module MCCplaca:ZCS18 (layer F.Cu)
@@
   (segment (start 267.284 100) (end 262.128 105.156) (width 12) (layer B.Cu) (net 48))
   (via (at 165.350917 113.217314) (size 1.7) (drill 0.6) (layers F.Cu B.Cu) (net 48))
-  (segment (start 212.555999 104.690001) (end 212.555999 104.690001) (width 12) (layer B.Cu) (net 48))
   (via (at 142.748 53.594) (size 1.7) (drill 0.6) (layers F.Cu B.Cu) (net 48))
   (segment (start 142.748 53.594) (end 140.208 53.594) (width 0.508) (layer F.Cu) (net 48))
@@
   (segment (start 165.350917 113.217314) (end 164.500918 112.367315) (width 0.508) (layer B.Cu) (net 48))
   (segment (start 164.500918 112.367315) (end 163.167315 112.367315) (width 0.508) (layer B.Cu) (net 48))
-  (segment (start 236.262001 104.690001) (end 212.555999 104.690001) (width 12) (layer B.Cu) (net 48))
-  (segment (start 236.728 105.156) (end 236.262001 104.690001) (width 12) (layer B.Cu) (net 48))
   (segment (start 174.498 108.458) (end 208.788 108.458) (width 9) (layer B.Cu) (net 48))
+  (segment (start 236.728 105.156) (end 213.021998 105.156) (width 12) (layer B.Cu) (net 48))
   (segment (start 166.624 33.02) (end 162.814 29.21) (width 0.508) (layer F.Cu) (net 49))
   (segment (start 168.91 24.9936) (end 174.652626 24.9936) (width 0.508) (layer F.Cu) (net 49))
