File: Hardware/Hall sensor/Cuk converter/KiCad/Mcc18.kicad_pcb (KiCad board)
At the start: 2 copper layers, 199.1 x 107.2 mm, 53 parts, among them Q1 IRFP4321PbF, U1 LTSP_25-NP, U2 DRIVER_(INEP), U3 LM7812_TO220, U4 Signals_MCC, U5 ZCS

Commit message: some zones fix
Routing:
- net GND: track 312.5 -> 315.1 mm, vias 10 -> 11
Changed lines of the file:
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@@
     (thickness 1.6)
     (drawings 8)
-    (tracks 549)
+    (tracks 552)
     (zones 0)
     (modules 53)
@@
     (user_trace_width 12)
     (trace_clearance 0.3048)
-    (zone_clearance 1.27)
+    (zone_clearance 0.3048)
     (zone_45_only no)
     (trace_min 0.508)
@@
   (segment (start 148.747 119.888) (end 146.715 121.92) (width 1) (layer B.Cu) (net 41) (status 20))
   (via (at 148.747 119.888) (size 1.7) (drill 0.6) (layers F.Cu B.Cu) (net 41))
-  (segment (start 148.747 121.090081) (end 145.377081 124.46) (width 1) (layer F.Cu) (net 41))
-  (segment (start 148.747 119.888) (end 148.747 121.090081) (width 1) (layer F.Cu) (net 41))
-  (segment (start 127.254 124.46) (end 119.126 132.588) (width 1) (layer F.Cu) (net 41))
-  (segment (start 145.377081 124.46) (end 127.254 124.46) (width 1) (layer F.Cu) (net 41))
   (via (at 157.226 111.252) (size 1.7) (drill 0.6) (layers F.Cu B.Cu) (net 41))
   (segment (start 112.522 66.294) (end 111.672001 65.444001) (width 1) (layer B.Cu) (net 41))
@@
   (segment (start 102.616 56.1825) (end 104.316 56.1825) (width 1) (layer F.Cu) (net 41) (status 10))
   (segment (start 111.672001 65.444001) (end 111.672001 63.666001) (width 1) (layer B.Cu) (net 41))
-  (via (at 115.824 133.858) (size 1.7) (drill 0.6) (layers F.Cu B.Cu) (net 41))
   (segment (start 94.996 96.012) (end 92.456 96.012) (width 0.508) (layer B.Cu) (net 41) (status 20))
   (segment (start 97.536 98.552) (end 94.996 96.012) (width 0.508) (layer B.Cu) (net 41))
@@
   (segment (start 136.144 56.388) (end 137.668 56.388) (width 1) (layer F.Cu) (net 41))
   (segment (start 137.668 56.388) (end 138.43 56.388) (width 1) (layer F.Cu) (net 41))
-  (segment (start 131.572 58.166) (end 132.842 56.896) (width 1) (layer F.Cu) (net 41))
-  (segment (start 132.842 56.896) (end 134.112 56.896) (width 1) (layer F.Cu) (net 41) (status 20))
-  (segment (start 131.572 60.96) (end 131.572 58.166) (width 1) (layer F.Cu) (net 41))
+  (segment (start 131.572 60.96) (end 130.556 60.198) (width 1) (layer F.Cu) (net 41))
   (segment (start 133.096 56.896) (end 134.112 56.896) (width 1) (layer F.Cu) (net 41))
   (segment (start 132.334 56.388) (end 132.588 56.388) (width 1) (layer F.Cu) (net 41))
@@
   (segment (start 157.226 111.252) (end 156.464 110.49) (width 0.508) (layer F.Cu) (net 41))
   (segment (start 156.464 110.49) (end 115.824 110.49) (width 0.508) (layer F.Cu) (net 41))
+  (via (at 130.556 60.198) (size 1.7) (drill 0.6) (layers F.Cu B.Cu) (net 41))
+  (segment (start 132.262 56.896) (end 134.112 56.896) (width 1) (layer B.Cu) (net 41))
+  (segment (start 130.556 58.602) (end 132.262 56.896) (width 1) (layer B.Cu) (net 41))
+  (segment (start 130.556 60.198) (end 130.556 58.602) (width 1) (layer B.Cu) (net 41))
+  (via (at 118.364 132.842) (size 1.7) (drill 0.6) (layers F.Cu B.Cu) (net 41))
+  (segment (start 119.213999 131.992001) (end 118.364 132.842) (width 1) (layer F.Cu) (net 41))
+  (segment (start 126.238 124.968) (end 119.213999 131.992001) (width 1) (layer F.Cu) (net 41))
+  (segment (start 145.542 124.968) (end 126.238 124.968) (width 1) (layer F.Cu) (net 41))
+  (segment (start 148.747 119.888) (end 148.747 121.763) (width 1) (layer F.Cu) (net 41))
+  (segment (start 148.747 121.763) (end 145.542 124.968) (width 1) (layer F.Cu) (net 41))
   (segment (start 144.78 125.73) (end 144.78 123.19) (width 1) (layer B.Cu) (net 42))
   (segment (start 144.78 123.19) (end 143.51 123.19) (width 1) (layer B.Cu) (net 42))
@@
     (polygon
       (pts
-        (xy 179.832 50.038) (xy 179.832 131.064) (xy 164.846 136.398) (xy 164.846 131.064) (xy 118.11 131.064)
+        (xy 179.832 50.038) (xy 179.832 136.398) (xy 164.846 136.398) (xy 127.508 136.398) (xy 118.11 126.746)
         (xy 118.11 50.038)
       )
@@
     )
   )
-  (zone (net 1) (net_name "Net-(U1-Pad3)") (layer B.Cu) (hatch none 0.508)
+  (zone (net 1) (net_name "Net-(U1-Pad3)") (layer B.Cu) (hatch full 0.508)
     (priority 10)
     (connect_pads yes (clearance 0.3048))
@@
     )
   )
-  (zone (net 35) (net_name "Net-(L1-Pad1)") (layer B.Cu) (hatch none 0.508)
+  (zone (net 35) (net_name "Net-(L1-Pad1)") (layer B.Cu) (hatch full 0.508)
     (priority 11)
     (connect_pads yes (clearance 0.3048))
@@
     (polygon
       (pts
-        (xy 179.832 50.038) (xy 179.832 136.398) (xy 164.846 136.398) (xy 164.846 131.064) (xy 118.11 131.064)
+        (xy 179.832 50.038) (xy 179.832 136.398) (xy 164.846 136.398) (xy 127.508 136.398) (xy 118.11 126.746)
         (xy 118.11 50.038)
       )
@@
   )
   (zone (net 41) (net_name GND) (layer F.Cu) (hatch edge 0.508)
+    (priority 4)
     (connect_pads yes (clearance 0.3048))
     (min_thickness 0.508)
@@
     (polygon
       (pts
-        (xy 50.038 39.878) (xy 116.586 39.878) (xy 116.586 49.022) (xy 118.11 50.546) (xy 118.11 131.064)
-        (xy 127.254 140.208) (xy 134.366 147.066) (xy 50.038 147.066)
+        (xy 50.038 39.878) (xy 116.586 39.878) (xy 116.586 49.022) (xy 118.11 50.546) (xy 118.11 109.22)
+        (xy 161.544 109.22) (xy 161.544 136.398) (xy 123.444 136.398) (xy 127.254 140.208) (xy 134.366 147.066)
+        (xy 50.038 147.066)
       )
     )

Commit message: minor fixes. GERBERS updated
Routing:
- net /-P_unfused: track 10.5 -> 19.8 mm
Changed lines of the file:
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@@
     (thickness 1.6)
     (drawings 8)
-    (tracks 552)
+    (tracks 553)
     (zones 0)
     (modules 53)
@@
   )
   (setup
-    (last_trace_width 1)
+    (last_trace_width 9)
     (user_trace_width 0.508)
     (user_trace_width 0.8)
@@
       (padsonsilk false)
       (subtractmaskfromsilk true)
-      (outputformat 1)
+      (outputformat 4)
       (mirror false)
       (drillshape 0)
       (scaleselection 1)
-      (outputdirectory GERBERS))
+      (outputdirectory PDF))
   )
   (net 0 "")
@@
     (arrow2b (pts (xy 38.608 39.878) (xy 39.194421 41.004504)))
   )
+  (segment (start 233.318 48.088) (end 240.094 54.864) (width 9) (layer F.Cu) (net 36))
   (segment (start 134.2136 58.928) (end 134.112 58.8264) (width 1) (layer B.Cu) (net 3) (status 30))
   (segment (start 137.668 58.928) (end 134.2136 58.928) (width 1) (layer B.Cu) (net 3) (status 30))
@@
   (segment (start 157.226 116.683) (end 154.94 116.683) (width 1) (layer B.Cu) (net 34) (status 30))
   (segment (start 240.202 54.972) (end 240.202 54.2994) (width 9) (layer B.Cu) (net 36) (status 30))
-  (segment (start 240.3544 54.6804) (end 233.426 47.752) (width 9) (layer B.Cu) (net 36) (status 30))
+  (segment (start 240.202 54.972) (end 233.426 48.196) (width 9) (layer B.Cu) (net 36))
   (segment (start 177.016 83.192) (end 177.038 83.214) (width 1) (layer F.Cu) (net 37) (status 30))
   (segment (start 177.016 76.454) (end 177.016 83.192) (width 1) (layer F.Cu) (net 37) (status 30))
