File: Hardware/Shunt sensor/Cuk converter/KiCad/Mcc18.sch (KiCad schematic (older format))
At the start: 60 parts, among them Q1 IRFP4321PbF, U1 INA240, U2 DRIVER_(INEP), U3 LM7812_TO220, U4 Signals_MCC, U5 ZCS, U6 INA211_DCK_6

Commit message: ok. Now it is on 25~50mils grid.
Parts:
- removed C11: 10uF, MCCplaca:C_0805_2012Metric_Pad1.29x1.40mm_HandSolder, symbol Device:C_Small
- removed C_INA211, C_INA240: 100n, MCCplaca:C_0805_2012Metric_Pad1.29x1.40mm_HandSolder, symbol Device:C_Small
- removed R107: 1R, Resistor_SMD:R_0805_2012Metric_Pad1.29x1.40mm_HandSolder, symbol Device:R_Small
- removed R_Ina211_Ref1, R_Ina211_SIG1, R_Ina240_REF1, R_Ina240_SIG1: ??, MCCplaca Shunt:R_0805_2012Metric_Pad1.29x1.40mm_HandSolder, symbol Device:R_Small
- added C? (x3): 100nF, MCC:C_0805_2012Metric_Pad1.29x1.40mm_HandSolder, symbol Device:C_Small
- added R? (x3): 0R, Resistor_SMD:R_0805_2012Metric_Pad1.29x1.40mm_HandSolder, symbol Device:R_Small
- added R? (x2): ??, Resistor_SMD:R_0805_2012Metric_Pad1.29x1.40mm_HandSolder, symbol Device:R_Small
- Rshunt: renamed from RShunt1; value R -> 500uR
- U1: symbol ina240_soic8:INA240 -> Mcc18-rescue:INA240-ina240_soic8
- U6: value INA211_DCK_6 -> INA211; symbol INA211BIDCKR:INA211_DCK_6 -> Mcc18-rescue:INA211_DCK_6-INA211BIDCKR
Connections:
- net labels added: INA211_OUT, INA240_OUT, Ip_sen+, Ip_sen-, Rs+, Rs-
- net labels removed: Ina240_REF, Ipanel_SIG, Ipanel_adc-, Shunt+, Shunt-
- wire segments 238 -> 249

Commit message: finished the first version
Parts:
- added R108: 0R, Jumper:SolderJumper-2_P1.3mm_Open_Pad1.0x1.5mm, symbol Device:R_Small
- C1, C11, C12: renamed from C?; footprint MCC:C_0805_2012Metric_Pad1.29x1.40mm_HandSolder -> MCCplaca Shunt:C_0805_2012Metric_Pad1.29x1.40mm_HandSolder
- R105, R106, R107: renamed from R?; footprint Resistor_SMD:R_0805_2012Metric_Pad1.29x1.40mm_HandSolder -> Jumper:SolderJumper-2_P1.3mm_Open_Pad1.0x1.5mm
- U1: symbol Mcc18-rescue:INA240-ina240_soic8 -> Mcc18-rescue:INA240-ina240_soic8-Mcc18-rescue
- U6: symbol Mcc18-rescue:INA211_DCK_6-INA211BIDCKR -> Mcc18-rescue:INA211_DCK_6-INA211BIDCKR-Mcc18-rescue
- gave numbers to parts that had none: 2
- renumbered Rshunt to Rshunt1
Connections:
- wire segments 249 -> 254
Changed lines of the file:
@@
 Vb_sen-
 $Comp
-L Mcc18-rescue:INA211_DCK_6-INA211BIDCKR U6
+L Mcc18-rescue:INA211_DCK_6-INA211BIDCKR-Mcc18-rescue U6
 U 1 1 5B11478B
 P 9975 6100
@@
 	2300 1400 5075 1400
 $Comp
-L Device:R Rshunt
+L Device:R Rshunt1
 U 1 1 5B4A6175
 P 2300 2650
-F 0 "Rshunt" H 2370 2696 50  0000 L CNN
+F 0 "Rshunt1" H 2370 2696 50  0000 L CNN
 F 1 "500uR" H 2370 2605 50  0000 L CNN
 F 2 "MCCplaca Shunt:PML100HZPJV0L5" V 2230 2650 50  0001 C CNN
@@
 Current Sensor\n
 $Comp
-L Mcc18-rescue:INA240-ina240_soic8 U1
+L Mcc18-rescue:INA240-ina240_soic8-Mcc18-rescue U1
 U 1 1 5B114902
 P 7725 5700
@@
 	7925 5950 7575 5950
 $Comp
-L power:GNDA #PWR?
+L power:GNDA #PWR0101
 U 1 1 5B34DCF0
 P 7450 6050
-F 0 "#PWR?" H 7450 5800 50  0001 C CNN
+F 0 "#PWR0101" H 7450 5800 50  0001 C CNN
 F 1 "GNDA" H 7455 5877 50  0000 C CNN
 F 2 "" H 7450 6050 50  0001 C CNN
@@
 $EndComp
 $Comp
-L Device:C_Small C?
+L Device:C_Small C11
 U 1 1 5B48C252
 P 8550 5625
-F 0 "C?" H 8642 5587 39  0000 L CNN
-F 1 "100nF" H 8642 5662 39  0000 L CNN
-F 2 "MCC:C_0805_2012Metric_Pad1.29x1.40mm_HandSolder" H 8550 5625 50  0001 C CNN
+F 0 "C11" H 8650 5550 39  0000 L CNN
+F 1 "100nF" H 8650 5600 39  0000 L CNN
+F 2 "MCCplaca Shunt:C_0805_2012Metric_Pad1.29x1.40mm_HandSolder" H 8550 5625 50  0001 C CNN
 F 3 "" H 8550 5625 50  0001 C CNN
 	1    8550 5625
 	1    0    0    1
 $EndComp
-$Comp
-L power:GND #PWR?
-U 1 1 5B48CFFA
-P 8550 5725
-F 0 "#PWR?" H 8550 5475 50  0001 C CNN
-F 1 "GND" H 8555 5552 50  0000 C CNN
-F 2 "" H 8550 5725 50  0001 C CNN
-F 3 "" H 8550 5725 50  0001 C CNN
-	1    8550 5725
-	-1   0    0    -1
-$EndComp
 Text Label 8325 6050 0    39   ~ 0
 INA240_OUT
 $Comp
-L power:+5VA #PWR?
+L power:+5VA #PWR0117
 U 1 1 5B575A82
 P 8400 5525
-F 0 "#PWR?" H 8400 5375 50  0001 C CNN
+F 0 "#PWR0117" H 8400 5375 50  0001 C CNN
 F 1 "+5VA" H 8415 5698 50  0000 C CNN
 F 2 "" H 8400 5525 50  0001 C CNN
@@
 	9250 5950 9475 5950
 $Comp
-L power:+5VA #PWR?
+L power:+5VA #PWR0118
 U 1 1 5B6360D0
 P 10125 5700
-F 0 "#PWR?" H 10125 5550 50  0001 C CNN
+F 0 "#PWR0118" H 10125 5550 50  0001 C CNN
 F 1 "+5VA" H 10140 5873 50  0000 C CNN
 F 2 "" H 10125 5700 50  0001 C CNN
@@
 $EndComp
 $Comp
-L Device:C_Small C?
+L Device:C_Small C12
 U 1 1 5B644DE0
 P 10300 5850
-F 0 "C?" H 10392 5812 39  0000 L CNN
+F 0 "C12" H 10392 5812 39  0000 L CNN
 F 1 "100nF" H 10392 5887 39  0000 L CNN
-F 2 "MCC:C_0805_2012Metric_Pad1.29x1.40mm_HandSolder" H 10300 5850 50  0001 C CNN
+F 2 "MCCplaca Shunt:C_0805_2012Metric_Pad1.29x1.40mm_HandSolder" H 10300 5850 50  0001 C CNN
 F 3 "" H 10300 5850 50  0001 C CNN
 	1    10300 5850
@@
 	10125 5950 10300 5950
 $Comp
-L power:GNDA #PWR?
+L power:GNDA #PWR0119
 U 1 1 5B69EBD7
 P 10300 6050
-F 0 "#PWR?" H 10300 5800 50  0001 C CNN
+F 0 "#PWR0119" H 10300 5800 50  0001 C CNN
 F 1 "GNDA" H 10305 5877 50  0000 C CNN
 F 2 "" H 10300 6050 50  0001 C CNN
@@
 INA211_OUT
 $Comp
-L Device:R_Small R?
+L Device:R_Small R106
 U 1 1 5B6DDB79
 P 9100 5725
-F 0 "R?" H 9041 5687 39  0000 R CNN
+F 0 "R106" H 9041 5687 39  0000 R CNN
 F 1 "0R" H 9041 5762 39  0000 R CNN
-F 2 "Resistor_SMD:R_0805_2012Metric_Pad1.29x1.40mm_HandSolder" H 9100 5725 50  0001 C CNN
+F 2 "Jumper:SolderJumper-2_P1.3mm_Open_Pad1.0x1.5mm" H 9100 5725 50  0001 C CNN
 F 3 "" H 9100 5725 50  0001 C CNN
 F 4 "1%" V 9175 5775 39  0001 C CNN "Tolerance"
@@
 $EndComp
 $Comp
-L Device:R_Small R?
+L Device:R_Small R105
 U 1 1 5B6EFB69
 P 9000 5725
-F 0 "R?" H 8941 5687 39  0000 R CNN
+F 0 "R105" H 8941 5687 39  0000 R CNN
 F 1 "0R" H 8941 5762 39  0000 R CNN
-F 2 "Resistor_SMD:R_0805_2012Metric_Pad1.29x1.40mm_HandSolder" H 9000 5725 50  0001 C CNN
+F 2 "Jumper:SolderJumper-2_P1.3mm_Open_Pad1.0x1.5mm" H 9000 5725 50  0001 C CNN
 F 3 "" H 9000 5725 50  0001 C CNN
 F 4 "1%" V 9075 5775 39  0001 C CNN "Tolerance"
@@
 	2400 7100 2400 7350
 $Comp
-L power:GNDA #PWR?
+L power:GNDA #PWR0120
 U 1 1 5B808DD3
 P 2950 7300
-F 0 "#PWR?" H 2950 7050 39  0001 C CNN
+F 0 "#PWR0120" H 2950 7050 39  0001 C CNN
 F 1 "GNDA" H 2955 7127 50  0000 C CNN
 F 2 "" H 2950 7300 50  0001 C CNN
@@
 $EndComp
 $Comp
-L Device:C_Small C?
+L Device:C_Small C1
 U 1 1 5B808F00
 P 2950 7050
-F 0 "C?" H 2858 7088 39  0000 R CNN
+F 0 "C1" H 2858 7088 39  0000 R CNN
 F 1 "100nF" H 2858 7013 39  0000 R CNN
-F 2 "MCC:C_0805_2012Metric_Pad1.29x1.40mm_HandSolder" H 2950 7050 50  0001 C CNN
+F 2 "MCCplaca Shunt:C_0805_2012Metric_Pad1.29x1.40mm_HandSolder" H 2950 7050 50  0001 C CNN
 F 3 "" H 2950 7050 50  0001 C CNN
 	1    2950 7050
@@
 	2950 7150 2950 7225
 $Comp
-L Device:R_Small R?
+L Device:R_Small R110
 U 1 1 5B817104
 P 3125 6850
-F 0 "R?" V 2953 6850 39  0000 C CNN
+F 0 "R110" V 2953 6850 39  0000 C CNN
 F 1 "??" V 3028 6850 39  0000 C CNN
 F 2 "Resistor_SMD:R_0805_2012Metric_Pad1.29x1.40mm_HandSolder" H 3125 6850 50  0001 C CNN
@@
 Connection ~ 10125 5950
 $Comp
-L Device:R_Small R?
+L Device:R_Small R109
 U 1 1 5BB245F0
 P 3125 7225
-F 0 "R?" V 3029 7225 39  0000 C CNN
+F 0 "R109" V 3029 7225 39  0000 C CNN
 F 1 "??" V 2954 7225 39  0000 C CNN
 F 2 "Resistor_SMD:R_0805_2012Metric_Pad1.29x1.40mm_HandSolder" H 3125 7225 50  0001 C CNN
@@
 Ip_sen-
 $Comp
-L Device:R_Small R?
+L Device:R_Small R107
 U 1 1 5BC9859D
 P 8950 5175
-F 0 "R?" H 8891 5137 39  0000 R CNN
-F 1 "0R" H 8891 5212 39  0000 R CNN
-F 2 "Resistor_SMD:R_0805_2012Metric_Pad1.29x1.40mm_HandSolder" H 8950 5175 50  0001 C CNN
+F 0 "R107" H 9150 5125 39  0000 R CNN
+F 1 "0R" H 9100 5200 39  0000 R CNN
+F 2 "Jumper:SolderJumper-2_P1.3mm_Open_Pad1.0x1.5mm" H 8950 5175 50  0001 C CNN
 F 3 "" H 8950 5175 50  0001 C CNN
 F 4 "1%" V 9025 5225 39  0001 C CNN "Tolerance"
@@
 $EndComp
 $Comp
-L power:GNDA #PWR?
+L power:GNDA #PWR0121
 U 1 1 5BC9865E
-P 8950 5275
-F 0 "#PWR?" H 8950 5025 50  0001 C CNN
-F 1 "GNDA" H 8955 5102 50  0000 C CNN
-F 2 "" H 8950 5275 50  0001 C CNN
-F 3 "" H 8950 5275 50  0001 C CNN
-	1    8950 5275
+P 8950 5300
+F 0 "#PWR0121" H 8950 5050 50  0001 C CNN
+F 1 "GNDA" H 8955 5127 50  0000 C CNN
+F 2 "" H 8950 5300 50  0001 C CNN
+F 3 "" H 8950 5300 50  0001 C CNN
+	1    8950 5300
 	-1   0    0    -1
 $EndComp
@@
 Wire Wire Line
 	8750 4950 9050 4950
-Wire Wire Line
-	8750 5050 8950 5050
 Wire Wire Line
 	8950 5050 8950 5075
@@
 Text Label 4845 5350 2    39   ~ 0
 Vp_sen-
+$Comp
+L Device:R_Small R108
+U 1 1 5B197291
+P 8850 5175
+F 0 "R108" H 8791 5137 39  0000 R CNN
+F 1 "0R" H 8791 5212 39  0000 R CNN
+F 2 "Jumper:SolderJumper-2_P1.3mm_Open_Pad1.0x1.5mm" H 8850 5175 50  0001 C CNN
+F 3 "" H 8850 5175 50  0001 C CNN
+F 4 "1%" V 8925 5225 39  0001 C CNN "Tolerance"
+	1    8850 5175
+	1    0    0    -1
+$EndComp
+Wire Wire Line
+	8750 5050 8850 5050
+Wire Wire Line
+	8850 5075 8850 5050
+Connection ~ 8850 5050
+Wire Wire Line
+	8850 5050 8950 5050
+Wire Wire Line
+	8850 5275 8950 5275
+Wire Wire Line
+	8950 5275 8950 5300
+Connection ~ 8950 5275
+$Comp
+L power:GNDA #PWR?
+U 1 1 5B21544E
+P 8550 5750
+F 0 "#PWR?" H 8550 5500 50  0001 C CNN
+F 1 "GNDA" H 8555 5577 50  0000 C CNN
+F 2 "" H 8550 5750 50  0001 C CNN
+F 3 "" H 8550 5750 50  0001 C CNN
+	1    8550 5750
+	1    0    0    -1
+$EndComp
+Wire Wire Line
+	8550 5725 8550 5750
 $EndSCHEMATC

Commit message: Added signals 3D in cuk PCB _Added signals 3D in signals component in MCCshunt Library._ _Added pin socket in the signals component_ _Added signals component in cuk converter PCB_ _Added MountingHoles to fix the signals PCB in thr cuk PCB_
Parts:
- added MK1: Mounting_Hole, MountingHole:MountingHole_2.2mm_M2_Pad, symbol Mechanical:Mounting_Hole
- U5: symbol ZCS:ZCS -> MCC18:ZCS-ZCS-Mcc18-rescue
Changed lines of the file:
@@
 	1750 6800 2400 6800
 $Comp
-L ZCS:ZCS U5
+L MCC18:ZCS-ZCS-Mcc18-rescue U5
 U 1 1 5B16184F
-P 1400 5000
-F 0 "U5" H 1531 5165 50  0000 C CNN
-F 1 "ZCS" H 1531 5074 50  0000 C CNN
-F 2 "MCCplaca:ZCS18" H 1400 5000 50  0001 C CNN
-F 3 "" H 1400 5000 50  0001 C CNN
-	1    1400 5000
+P 1300 5000
+F 0 "U5" H 1431 5165 50  0000 C CNN
+F 1 "ZCS" H 1431 5074 50  0000 C CNN
+F 2 "MCCplaca:ZCS18" H 1300 5000 50  0001 C CNN
+F 3 "" H 1300 5000 50  0001 C CNN
+	1    1300 5000
 	1    0    0    -1
 $EndComp
@@
 Connection ~ 8950 5275
 $Comp
-L power:GNDA #PWR?
+L power:GNDA #PWR0102
 U 1 1 5B21544E
 P 8550 5750
-F 0 "#PWR?" H 8550 5500 50  0001 C CNN
+F 0 "#PWR0102" H 8550 5500 50  0001 C CNN
 F 1 "GNDA" H 8555 5577 50  0000 C CNN
 F 2 "" H 8550 5750 50  0001 C CNN
@@
 Wire Wire Line
 	8550 5725 8550 5750
+$Comp
+L Mechanical:Mounting_Hole MK1
+U 1 1 5B14A5CB
+P 1150 4025
+F 0 "MK1" H 1250 4071 50  0000 L CNN
+F 1 "Mounting_Hole" H 1250 3980 50  0000 L CNN
+F 2 "MountingHole:MountingHole_2.2mm_M2_Pad" H 1150 4025 50  0001 C CNN
+F 3 "" H 1150 4025 50  0001 C CNN
+	1    1150 4025
+	1    0    0    -1
+$EndComp
 $EndSCHEMATC
