File: Hardware/Shunt sensor/Cuk converter/KiCad/Mcc18.kicad_pcb (KiCad board)
At the start: 2 copper layers, 199.1 x 107.2 mm, 62 parts, among them Q1 IRFP4321PbF, U1 INA240, U2 DRIVER_(INEP), U3 LM7812_TO220, U4 Signals_MCC, U5 ZCS, U6 INA211

Commit message: Updated fabrication outputs _Updated shunt signals PDF schematic,PDF PCB, GERBER PCB,Drill PCB_ _Updated shunt cuk PDF schematic,PDF PCB, GERBER PCB,Drill PCB_ _Updated hall signals PDF schematic,PDF PCB, GERBER PCB,Drill PCB_ _Updated hall cuk PDF schematic,PDF PCB, GERBER PCB,Drill PCB_
Routing:
- net /Vp_sen-: track 166.0 -> 161.7 mm
- net /Vp_sen+: track 168.6 -> 164.5 mm
Changed lines of the file:
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@@
     (thickness 1.6)
     (drawings 8)
-    (tracks 675)
+    (tracks 671)
     (zones 0)
     (modules 62)
@@
   (segment (start 92.075 140.716) (end 91.948 140.843) (width 0.508) (layer B.Cu) (net 50) (status 30))
   (segment (start 105.81 108.966) (end 105.41 108.966) (width 0.635) (layer F.Cu) (net 51) (status 40000))
-  (segment (start 112.386735 45.5041) (end 110.0201 47.870735) (width 0.635) (layer F.Cu) (net 51) (status 40000))
-  (segment (start 129.48064 45.5041) (end 112.386735 45.5041) (width 0.635) (layer F.Cu) (net 51) (status 40000))
-  (segment (start 132.02064 48.0441) (end 129.48064 45.5041) (width 0.635) (layer F.Cu) (net 51) (status 40000))
-  (segment (start 186.432 65.532) (end 185.2509 66.7131) (width 0.635) (layer F.Cu) (net 51) (status 40000))
-  (segment (start 186.4845 65.532) (end 186.432 65.532) (width 0.635) (layer F.Cu) (net 51) (status 40000))
+  (segment (start 103.6099 108.1659) (end 104.41 108.966) (width 0.635) (layer F.Cu) (net 51) (status 40000))
+  (segment (start 102.8319 108.65264) (end 103.31864 108.1659) (width 0.635) (layer F.Cu) (net 51) (status 40000))
+  (segment (start 182.3339 64.57536) (end 182.3339 54.3179) (width 0.635) (layer F.Cu) (net 51) (status 40000))
   (segment (start 185.2509 66.7131) (end 184.47164 66.7131) (width 0.635) (layer F.Cu) (net 51) (status 40000))
+  (segment (start 182.3339 54.3179) (end 182.23644 54.3179) (width 0.635) (layer F.Cu) (net 51))
+  (segment (start 186.4845 65.532) (end 186.432 65.532) (width 0.635) (layer F.Cu) (net 51))
+  (segment (start 113.4999 48.0441) (end 110.0201 51.5239) (width 0.635) (layer F.Cu) (net 51) (status 40000))
+  (segment (start 186.432 65.532) (end 185.2509 66.7131) (width 0.635) (layer F.Cu) (net 51) (status 40000))
+  (segment (start 107.9881 106.99336) (end 107.9881 109.53336) (width 0.635) (layer F.Cu) (net 51) (status 40000))
   (segment (start 184.47164 66.7131) (end 182.3339 64.57536) (width 0.635) (layer F.Cu) (net 51) (status 40000))
-  (segment (start 182.3339 64.57536) (end 182.3339 54.3179) (width 0.635) (layer F.Cu) (net 51) (status 40000))
-  (segment (start 182.3339 54.3179) (end 182.23644 54.3179) (width 0.635) (layer F.Cu) (net 51) (status 40000))
   (segment (start 182.23644 54.3179) (end 175.96264 48.0441) (width 0.635) (layer F.Cu) (net 51) (status 40000))
-  (segment (start 175.96264 48.0441) (end 132.02064 48.0441) (width 0.635) (layer F.Cu) (net 51) (status 40000))
-  (segment (start 105.41 108.966) (end 104.41 108.966) (width 0.635) (layer F.Cu) (net 51) (status 40000))
-  (segment (start 104.41 108.966) (end 103.6099 108.1659) (width 0.635) (layer F.Cu) (net 51) (status 40000))
-  (segment (start 103.6099 108.1659) (end 103.31864 108.1659) (width 0.635) (layer F.Cu) (net 51) (status 40000))
-  (segment (start 103.31864 108.1659) (end 102.8319 108.65264) (width 0.635) (layer F.Cu) (net 51) (status 40000))
-  (segment (start 102.8319 108.65264) (end 102.8319 109.78736) (width 0.635) (layer F.Cu) (net 51) (status 40000))
-  (segment (start 102.8319 109.78736) (end 103.82664 110.7821) (width 0.635) (layer F.Cu) (net 51) (status 40000))
-  (segment (start 103.82664 110.7821) (end 106.73936 110.7821) (width 0.635) (layer F.Cu) (net 51) (status 40000))
-  (segment (start 106.73936 110.7821) (end 107.9881 109.53336) (width 0.635) (layer F.Cu) (net 51) (status 40000))
-  (segment (start 107.9881 109.53336) (end 107.9881 106.99336) (width 0.635) (layer F.Cu) (net 51) (status 40000))
-  (segment (start 110.0201 47.870735) (end 110.0201 104.96136) (width 0.635) (layer F.Cu) (net 51) (status 40000))
+  (segment (start 103.31864 108.1659) (end 103.6099 108.1659) (width 0.635) (layer F.Cu) (net 51))
+  (segment (start 175.96264 48.0441) (end 113.4999 48.0441) (width 0.635) (layer F.Cu) (net 51) (status 40000))
+  (segment (start 110.0201 51.5239) (end 110.0201 104.96136) (width 0.635) (layer F.Cu) (net 51) (status 40000))
+  (segment (start 107.9881 109.53336) (end 106.73936 110.7821) (width 0.635) (layer F.Cu) (net 51) (status 40000))
+  (segment (start 106.73936 110.7821) (end 103.82664 110.7821) (width 0.635) (layer F.Cu) (net 51) (status 40000))
+  (segment (start 104.41 108.966) (end 105.41 108.966) (width 0.635) (layer F.Cu) (net 51))
   (segment (start 110.0201 104.96136) (end 107.9881 106.99336) (width 0.635) (layer F.Cu) (net 51) (status 40000))
+  (segment (start 103.82664 110.7821) (end 102.8319 109.78736) (width 0.635) (layer F.Cu) (net 51) (status 40000))
+  (segment (start 102.8319 109.78736) (end 102.8319 108.65264) (width 0.635) (layer F.Cu) (net 51) (status 40000))
   (segment (start 186.4845 68.834) (end 186.4845 68.7815) (width 0.635) (layer F.Cu) (net 52) (status 40030))
+  (segment (start 104.41 106.426) (end 105.41 106.426) (width 0.635) (layer F.Cu) (net 52))
+  (segment (start 103.6099 107.2261) (end 104.41 106.426) (width 0.635) (layer F.Cu) (net 52) (status 40000))
+  (segment (start 102.92936 107.2261) (end 103.6099 107.2261) (width 0.635) (layer F.Cu) (net 52) (status 40000))
+  (segment (start 181.3941 54.80464) (end 175.57336 48.9839) (width 0.635) (layer F.Cu) (net 52) (status 40000))
+  (segment (start 181.3941 64.96464) (end 181.3941 54.80464) (width 0.635) (layer F.Cu) (net 52) (status 40000))
   (segment (start 184.08236 67.6529) (end 181.3941 64.96464) (width 0.635) (layer F.Cu) (net 52) (status 40000))
   (segment (start 185.2509 67.6529) (end 184.08236 67.6529) (width 0.635) (layer F.Cu) (net 52) (status 40000))
   (segment (start 186.432 68.834) (end 185.2509 67.6529) (width 0.635) (layer F.Cu) (net 52) (status 40000))
-  (segment (start 186.4845 68.834) (end 186.432 68.834) (width 0.635) (layer F.Cu) (net 52) (status 40000))
-  (segment (start 181.3941 54.80464) (end 175.57336 48.9839) (width 0.635) (layer F.Cu) (net 52) (status 40000))
-  (segment (start 175.57336 48.9839) (end 131.63136 48.9839) (width 0.635) (layer F.Cu) (net 52) (status 40000))
-  (segment (start 181.3941 64.96464) (end 181.3941 54.80464) (width 0.635) (layer F.Cu) (net 52) (status 40000))
-  (segment (start 131.63136 48.9839) (end 129.09136 46.4439) (width 0.635) (layer F.Cu) (net 52) (status 40000))
-  (segment (start 129.09136 46.4439) (end 112.97064 46.4439) (width 0.635) (layer F.Cu) (net 52) (status 40000))
-  (segment (start 112.97064 46.4439) (end 110.9599 48.45464) (width 0.635) (layer F.Cu) (net 52) (status 40000))
-  (segment (start 104.41 106.426) (end 103.6099 107.2261) (width 0.635) (layer F.Cu) (net 52) (status 40000))
-  (segment (start 105.41 106.426) (end 104.41 106.426) (width 0.635) (layer F.Cu) (net 52) (status 40000))
-  (segment (start 103.6099 107.2261) (end 102.92936 107.2261) (width 0.635) (layer F.Cu) (net 52) (status 40000))
-  (segment (start 102.92936 107.2261) (end 101.8921 108.26336) (width 0.635) (layer F.Cu) (net 52) (status 40000))
-  (segment (start 101.8921 108.26336) (end 101.8921 110.17664) (width 0.635) (layer F.Cu) (net 52) (status 40000))
-  (segment (start 101.8921 110.17664) (end 103.43736 111.7219) (width 0.635) (layer F.Cu) (net 52) (status 40000))
-  (segment (start 103.43736 111.7219) (end 107.12864 111.7219) (width 0.635) (layer F.Cu) (net 52) (status 40000))
-  (segment (start 107.12864 111.7219) (end 108.9279 109.92264) (width 0.635) (layer F.Cu) (net 52) (status 40000))
-  (segment (start 108.9279 109.92264) (end 108.9279 107.38264) (width 0.635) (layer F.Cu) (net 52) (status 40000))
+  (segment (start 175.57336 48.9839) (end 113.8301 48.9839) (width 0.635) (layer F.Cu) (net 52) (status 40000))
+  (segment (start 110.9599 51.8541) (end 110.9599 105.35064) (width 0.635) (layer F.Cu) (net 52) (status 40000))
   (segment (start 110.9599 105.35064) (end 108.9279 107.38264) (width 0.635) (layer F.Cu) (net 52) (status 40000))
-  (segment (start 110.9599 48.45464) (end 110.9599 105.35064) (width 0.635) (layer F.Cu) (net 52) (status 40000))
+  (segment (start 113.8301 48.9839) (end 110.9599 51.8541) (width 0.635) (layer F.Cu) (net 52) (status 40000))
+  (segment (start 103.43736 111.7219) (end 101.8921 110.17664) (width 0.635) (layer F.Cu) (net 52) (status 40000))
+  (segment (start 101.8921 110.17664) (end 101.8921 108.26336) (width 0.635) (layer F.Cu) (net 52) (status 40000))
+  (segment (start 186.4845 68.834) (end 186.432 68.834) (width 0.635) (layer F.Cu) (net 52))
+  (segment (start 108.9279 107.38264) (end 108.9279 109.92264) (width 0.635) (layer F.Cu) (net 52) (status 40000))
+  (segment (start 108.9279 109.92264) (end 107.12864 111.7219) (width 0.635) (layer F.Cu) (net 52) (status 40000))
+  (segment (start 107.12864 111.7219) (end 103.43736 111.7219) (width 0.635) (layer F.Cu) (net 52) (status 40000))
+  (segment (start 101.8921 108.26336) (end 102.92936 107.2261) (width 0.635) (layer F.Cu) (net 52) (status 40000))
   (segment (start 107.9255 82.7659) (end 108.458 83.2984) (width 0.635) (layer F.Cu) (net 53) (status 40000))
   (segment (start 107.2101 82.7659) (end 107.9255 82.7659) (width 0.635) (layer F.Cu) (net 53) (status 40000))
