File: Hardware/Shunt sensor/Signals/Signal.sch (KiCad schematic (older format))
At the start: 22 parts, among them Q1 Q_NPN_Darlington_BEC, U1 Signals_MCC, U2 LM324, U3 INA826_D_8

Commit message: shunt signals updated
Parts:
- removed R? (x2): ??, Resistor_SMD:R_0805_2012Metric_Pad1.29x1.40mm_HandSolder, symbol Device:R_US
- added R11: ??, Resistor_SMD:R_0805_2012Metric_Pad1.29x1.40mm_HandSolder, symbol Device:R_US
- gave numbers to parts that had none: 2
Connections:
- wire segments 93 -> 97
Other:
- moved on the sheet: U2D
Changed lines of the file:
@@
-$EndComp
-$Comp
-L power:+5VA #PWR0105
-U 1 1 5AE45329
-P 2550 2125
-F 0 "#PWR0105" H 2550 1975 50  0001 C CNN
-F 1 "+5VA" H 2565 2298 50  0000 C CNN
-F 2 "" H 2550 2125 50  0001 C CNN
-F 3 "" H 2550 2125 50  0001 C CNN
-	1    2550 2125
-	1    0    0    -1
 $EndComp
 $Comp
@@
 Wire Wire Line
 	3100 2175 3300 2175
-Wire Wire Line
-	2900 2175 2550 2175
-Wire Wire Line
-	2550 2175 2550 2275
-Connection ~ 2550 2175
-Wire Wire Line
-	2550 2125 2550 2175
 $Comp
 L Amplifier_Operational:LM324 U2
@@
 L Amplifier_Operational:LM324 U2
 U 4 1 5AF5A2A4
-P 3650 1400
-F 0 "U2" H 3675 1600 50  0000 L CNN
-F 1 "LM324" H 3675 1525 50  0000 L CNN
-F 2 "Package_SO:SOIC-14_3.9x8.7mm_P1.27mm" H 3600 1500 50  0001 C CNN
-F 3 "http://www.ti.com/lit/ds/symlink/lm124-n.pdf" H 3700 1600 50  0001 C CNN
-	4    3650 1400
+P 4425 925
+F 0 "U2" H 4450 1125 50  0000 L CNN
+F 1 "LM324" H 4450 1050 50  0000 L CNN
+F 2 "Package_SO:SOIC-14_3.9x8.7mm_P1.27mm" H 4375 1025 50  0001 C CNN
+F 3 "http://www.ti.com/lit/ds/symlink/lm124-n.pdf" H 4475 1125 50  0001 C CNN
+	4    4425 925
 	1    0    0    -1
 $EndComp
@@
 	3250 825  3350 825
 Wire Wire Line
-	3250 1300 3350 1300
+	4025 825  4125 825
 $Comp
 L power:GNDA #PWR0120
@@
 L power:GNDA #PWR0121
 U 1 1 5AF5F864
-P 3250 1300
-F 0 "#PWR0121" H 3250 1050 50  0001 C CNN
-F 1 "GNDA" H 3255 1127 50  0000 C CNN
-F 2 "" H 3250 1300 50  0001 C CNN
-F 3 "" H 3250 1300 50  0001 C CNN
-	1    3250 1300
+P 4025 825
+F 0 "#PWR0121" H 4025 575 50  0001 C CNN
+F 1 "GNDA" H 4030 652 50  0000 C CNN
+F 2 "" H 4025 825 50  0001 C CNN
+F 3 "" H 4025 825 50  0001 C CNN
+	1    4025 825
 	1    0    0    -1
 $EndComp
@@
 	3950 1150 3950 925
 Wire Wire Line
-	3350 1500 3350 1625
-Wire Wire Line
-	3350 1625 3950 1625
-Wire Wire Line
-	3950 1625 3950 1400
+	4125 1025 4125 1150
+Wire Wire Line
+	4125 1150 4725 1150
+Wire Wire Line
+	4725 1150 4725 925
 $Comp
 L MCC18:Signals_MCC-MCC18-Mcc18-rescue-Mcc18-rescue-Mcc18-rescue-Mcc18-rescue U1
@@
 Text Label 1275 3900 2    39   ~ 0
 Vpanel_Ref
-Wire Wire Line
-	2150 3900 1725 3900
 Text Label 1275 4500 2    39   ~ 0
 Vpanel_SIG
@@
 	4600 3925 4600 3900
 $Comp
-L Device:R_US R?
-U 1 1 5B1193A4
-P 1550 3900
-F 0 "R?" V 1625 3900 50  0000 C CNN
-F 1 "??" V 1700 3900 50  0000 C CNN
-F 2 "Resistor_SMD:R_0805_2012Metric_Pad1.29x1.40mm_HandSolder" V 1590 3890 50  0001 C CNN
-F 3 "~" H 1550 3900 50  0001 C CNN
-	1    1550 3900
-	0    1    1    0
-$EndComp
-$Comp
-L Device:R_US R?
+L Device:R_US R9
 U 1 1 5B11947E
-P 1725 4050
-F 0 "R?" V 1800 4050 50  0000 C CNN
-F 1 "??" V 1875 4050 50  0000 C CNN
-F 2 "Resistor_SMD:R_0805_2012Metric_Pad1.29x1.40mm_HandSolder" V 1765 4040 50  0001 C CNN
-F 3 "~" H 1725 4050 50  0001 C CNN
-	1    1725 4050
+P 1725 3700
+F 0 "R9" V 1800 3700 50  0000 C CNN
+F 1 "??" V 1875 3700 50  0000 C CNN
+F 2 "Resistor_SMD:R_0805_2012Metric_Pad1.29x1.40mm_HandSolder" V 1765 3690 50  0001 C CNN
+F 3 "~" H 1725 3700 50  0001 C CNN
+	1    1725 3700
 	-1   0    0    1
 $EndComp
-Connection ~ 1725 3900
-Wire Wire Line
-	1725 3900 1700 3900
-Wire Wire Line
-	1700 4500 1725 4500
-$Comp
-L power:GNDA #PWR?
+$Comp
+L power:GNDA #PWR0109
 U 1 1 5B11BAB1
-P 1725 4250
-F 0 "#PWR?" H 1725 4000 50  0001 C CNN
-F 1 "GNDA" H 1730 4077 50  0000 C CNN
-F 2 "" H 1725 4250 50  0001 C CNN
-F 3 "" H 1725 4250 50  0001 C CNN
-	1    1725 4250
-	1    0    0    -1
-$EndComp
-Wire Wire Line
-	1725 4250 1725 4200
-$Comp
-L Device:R_US R?
-U 1 1 5B11E06E
-P 1550 4500
-F 0 "R?" V 1625 4500 50  0000 C CNN
-F 1 "??" V 1700 4500 50  0000 C CNN
-F 2 "Resistor_SMD:R_0805_2012Metric_Pad1.29x1.40mm_HandSolder" V 1590 4490 50  0001 C CNN
-F 3 "~" H 1550 4500 50  0001 C CNN
-	1    1550 4500
-	0    1    1    0
-$EndComp
-$Comp
-L Device:R_US R?
+P 1725 3500
+F 0 "#PWR0109" H 1725 3250 50  0001 C CNN
+F 1 "GNDA" H 1730 3327 50  0000 C CNN
+F 2 "" H 1725 3500 50  0001 C CNN
+F 3 "" H 1725 3500 50  0001 C CNN
+	1    1725 3500
+	-1   0    0    1
+$EndComp
+$Comp
+L Device:R_US R10
 U 1 1 5B11E0CA
 P 1725 4650
-F 0 "R?" V 1800 4650 50  0000 C CNN
+F 0 "R10" V 1800 4650 50  0000 C CNN
 F 1 "??" V 1875 4650 50  0000 C CNN
 F 2 "Resistor_SMD:R_0805_2012Metric_Pad1.29x1.40mm_HandSolder" V 1765 4640 50  0001 C CNN
 F 3 "~" H 1725 4650 50  0001 C CNN
 	1    1725 4650
-	-1   0    0    1
-$EndComp
-Connection ~ 1725 4500
-Wire Wire Line
-	1725 4500 2150 4500
-$Comp
-L power:GNDA #PWR?
+	1    0    0    1
+$EndComp
+$Comp
+L power:GNDA #PWR0110
 U 1 1 5B11E122
 P 1725 4825
-F 0 "#PWR?" H 1725 4575 50  0001 C CNN
+F 0 "#PWR0110" H 1725 4575 50  0001 C CNN
 F 1 "GNDA" H 1730 4652 50  0000 C CNN
 F 2 "" H 1725 4825 50  0001 C CNN
@@
 	1725 4825 1725 4800
 Wire Wire Line
-	1400 4500 950  4500
-Wire Wire Line
-	1400 3900 950  3900
+	1725 3550 1725 3500
+Wire Wire Line
+	1725 3850 1725 3900
+Connection ~ 1725 3900
+Wire Wire Line
+	1725 3900 1800 3900
+$Comp
+L Device:R_US R11
+U 1 1 5B14056E
+P 1800 4175
+F 0 "R11" V 1875 4175 50  0000 C CNN
+F 1 "??" V 1950 4175 50  0000 C CNN
+F 2 "Resistor_SMD:R_0805_2012Metric_Pad1.29x1.40mm_HandSolder" V 1840 4165 50  0001 C CNN
+F 3 "~" H 1800 4175 50  0001 C CNN
+	1    1800 4175
+	-1   0    0    1
+$EndComp
+Wire Wire Line
+	1800 4025 1800 3900
+Connection ~ 1800 3900
+Wire Wire Line
+	1800 3900 2150 3900
+Wire Wire Line
+	1800 4325 1800 4500
+Wire Wire Line
+	1800 4500 2150 4500
+Wire Wire Line
+	950  3900 1725 3900
+Wire Wire Line
+	950  4500 1725 4500
+Connection ~ 1800 4500
+Connection ~ 1725 4500
+Wire Wire Line
+	1725 4500 1800 4500
+$Comp
+L power:+5VA #PWR0111
+U 1 1 5B17F39D
+P 3550 600
+F 0 "#PWR0111" H 3550 450 50  0001 C CNN
+F 1 "+5VA" H 3565 773 50  0000 C CNN
+F 2 "" H 3550 600 50  0001 C CNN
+F 3 "" H 3550 600 50  0001 C CNN
+	1    3550 600
+	1    0    0    -1
+$EndComp
+Wire Wire Line
+	3550 600  3550 625
+$Comp
+L power:+5VA #PWR0105
+U 1 1 5B182471
+P 2550 2125
+F 0 "#PWR0105" H 2550 1975 50  0001 C CNN
+F 1 "+5VA" H 2565 2298 50  0000 C CNN
+F 2 "" H 2550 2125 50  0001 C CNN
+F 3 "" H 2550 2125 50  0001 C CNN
+	1    2550 2125
+	1    0    0    -1
+$EndComp
+Wire Wire Line
+	2550 2125 2550 2275
+$Comp
+L power:+5VA #PWR0112
+U 1 1 5B1854FA
+P 2825 2150
+F 0 "#PWR0112" H 2825 2000 50  0001 C CNN
+F 1 "+5VA" H 2840 2323 50  0000 C CNN
+F 2 "" H 2825 2150 50  0001 C CNN
+F 3 "" H 2825 2150 50  0001 C CNN
+	1    2825 2150
+	1    0    0    -1
+$EndComp
+Wire Wire Line
+	2825 2150 2825 2175
+Wire Wire Line
+	2825 2175 2900 2175
+$Comp
+L power:+5VA #PWR0113
+U 1 1 5B18E263
+P 4325 625
+F 0 "#PWR0113" H 4325 475 50  0001 C CNN
+F 1 "+5VA" H 4340 798 50  0000 C CNN
+F 2 "" H 4325 625 50  0001 C CNN
+F 3 "" H 4325 625 50  0001 C CNN
+	1    4325 625
+	1    0    0    -1
+$EndComp
 $EndSCHEMATC
