File: Hardware/Hall_sensor/Signals/Signal.kicad_pcb (KiCad board)
At the start: 2 copper layers, 72.6 x 35.6 mm, 46 parts, among them Q1 Q_NPN_Darlington_BEC, U1 Signals_MCC, U2 LM324, U3 LM324, U4 LM324

Commit message: fixed and created all Fabrication files
Parts:
- moved R33 1.27 mm to (59.9, 24.4)
- moved R32 1.25 mm to (31.5, 23.0)
- moved Q1 1.14 mm to (72.6, 25.9)
- moved R31 0.50 mm to (31.5, 17.8)
- moved R35 0.19 mm to (27.2, 20.6)
Routing:
- net GNDA: track 182.4 -> 194.0 mm, vias 6 -> 8
- net +5VA: track 108.0 -> 109.1 mm
- net Net-(Q1-Pad3): track 2.05 -> 2.98 mm
- net /Ipanel_SIG: track 22.0 -> 22.9 mm
- net /Vpanel_SIG: track 30.4 -> 31.2 mm
- net Net-(R33-Pad1): track 19.9 -> 20.7 mm
- net /Ipanel_Ref: track 18.7 -> 19.3 mm
- net /Vpanel_Ref: track 22.4 -> 23.1 mm
- net Net-(Q1-Pad1): track 7.54 -> 6.90 mm
- added copper zone on F.Cu, net GNDA
