File: Hardware/Shunt_sensor/Signals/Signal.kicad_pcb (KiCad board)
At the start: 2 copper layers, 55.4 x 29.5 mm, 21 parts, among them Q1 Q_NPN_Darlington_BEC, U1 Signals_MCC, U2 LM324, U3 INA826_D_8

Commit message: fixed and created all Fabrication files
Parts:
- moved R4 1.47 mm to (68.1, 22.9)
- moved Q1 1.44 mm to (71.1, 25.9)
- moved R2 1.37 mm to (69.6, 16.5)
- moved U1 1.27 mm to (28.4, 6.35)
Routing:
- net GNDA: track 172.3 -> 183.7 mm, vias 6 -> 8
- net /Vpanel_SIG: track 8.37 -> 11.8 mm
- net /Vpanel_Ref: track 8.45 -> 11.6 mm
- net /BatOVInterrupt: track 17.4 -> 20.2 mm
- net /Vbat: track 16.2 -> 14.1 mm
- net /Vbat_SIG_IN: track 2.61 -> 4.64 mm
- net Net-(Q1-Pad1): track 6.86 -> 8.33 mm
- net /Vpanel: track 6.35 -> 7.67 mm
- net +5VA: track 80.9 -> 82.2 mm
- net Net-(Q1-Pad3): track 2.05 -> 2.93 mm
- net /Ipanel_Ref: track 0.86 -> 0.00 mm
- net /PWM: track 2.64 -> 3.38 mm
- added copper zone on F.Cu, net GNDA
Other:
- board size 55.4 x 29.5 mm -> 55.4 x 30.7 mm
