File: Hardware/Hall_sensor/Cuk_converter/KiCad/Mcc18.sch (KiCad schematic (older format))
At the start: 53 parts, among them Q1 IRFP4321PbF, U1 LTSP_25-NP, U2 DRIVER_(INEP), U3 LM7812_TO220, U4 Signals_MCC, U5 ZCS

Commit message: Added trak between Shunt and Inductor
Other:
- moved on the sheet: U3
