File: Hardware/Shunt_sensor/Cuk_converter/KiCad/_saved_Mcc18.sch (KiCad schematic (older format))
At the start: 61 parts, among them Q1 IRFP4321PbF, U1 INA240, U2 DRIVER_(INEP), U3 LM7812_TO220, U4 Signals_MCC, U5 ZCS

Commit message: Copper Clearence fixed
Parts:
- U1: symbol Mcc18-rescue:INA240-ina240_soic8-Mcc18-rescue-Mcc18-rescue -> Mcc18-rescue:INA240-ina240_soic8-Mcc18-rescue-Mcc18-rescue-Mcc18-rescue
Connections:
- wire segments 252 -> 253
Changed lines of the file:
@@
 Current Sensor\n
 $Comp
-L Mcc18-rescue:INA240-ina240_soic8-Mcc18-rescue-Mcc18-rescue U1
+L Mcc18-rescue:INA240-ina240_soic8-Mcc18-rescue-Mcc18-rescue-Mcc18-rescue U1
 U 1 1 5B114902
 P 7725 5700
@@
 Text Label 8325 6050 0    39   ~ 0
 INA240_OUT
-$Comp
-L power:+5VA #PWR0117
-U 1 1 5B575A82
-P 8400 5525
-F 0 "#PWR0117" H 8400 5375 50  0001 C CNN
-F 1 "+5VA" H 8415 5698 50  0000 C CNN
-F 2 "" H 8400 5525 50  0001 C CNN
-F 3 "" H 8400 5525 50  0001 C CNN
-	1    8400 5525
-	1    0    0    -1
-$EndComp
 $Comp
 L Device:R_Small R105
@@
 Wire Wire Line
 	8400 5525 8400 5950
-Connection ~ 8400 5525
 Wire Wire Line
 	3225 6850 3350 6850
@@
 	10200 5600 10400 5600
 $Comp
-L power:GNDA #PWR0118
+L power:GNDA #PWR0117
 U 1 1 5B293664
 P 9800 6000
-F 0 "#PWR0118" H 9800 5750 39  0001 C CNN
+F 0 "#PWR0117" H 9800 5750 39  0001 C CNN
 F 1 "GNDA" H 9900 5825 50  0000 R CNN
 F 2 "" H 9800 6000 50  0001 C CNN
@@
 $EndComp
 $Comp
-L power:GND #PWR0119
+L power:GND #PWR0118
 U 1 1 5B29366A
 P 10200 6000
-F 0 "#PWR0119" H 10200 5750 50  0001 C CNN
+F 0 "#PWR0118" H 10200 5750 50  0001 C CNN
 F 1 "GND" H 10205 5827 50  0000 C CNN
 F 2 "" H 10200 6000 50  0001 C CNN
@@
 	10400 5600 10550 5600
 $Comp
-L power:+5VA #PWR0122
-U 1 1 5B29367F
-P 9700 5475
-F 0 "#PWR0122" H 9700 5325 50  0001 C CNN
-F 1 "+5VA" H 9715 5603 50  0000 L CNN
-F 2 "" H 9700 5475 50  0001 C CNN
-F 3 "" H 9700 5475 50  0001 C CNN
-	1    9700 5475
-	1    0    0    -1
-$EndComp
-$Comp
-L power:+5V #PWR0123
+L power:+5V #PWR0119
 U 1 1 5B293685
 P 10400 5500
-F 0 "#PWR0123" H 10400 5350 50  0001 C CNN
+F 0 "#PWR0119" H 10400 5350 50  0001 C CNN
 F 1 "+5V" H 10415 5673 50  0000 C CNN
 F 2 "" H 10400 5500 50  0001 C CNN
@@
 $EndComp
 Wire Wire Line
-	9700 5475 9700 5600
-Wire Wire Line
-	9700 5600 9800 5600
+	8800 5600 8800 5525
+Wire Wire Line
+	8800 5525 8550 5525
+Wire Wire Line
+	8800 5600 9800 5600
+Connection ~ 8550 5525
 $EndSCHEMATC
