File: Hardware/Shunt_sensor/Cuk_converter/KiCad/Mcc18.sch (KiCad schematic (older format))
At the start: 62 parts, among them Q1 IRFP4321PbF, U1 INA240, U2 DRIVER_(INEP), U3 LM7812_TO220, U4 Signals_MCC, U5 ZCS, U6 INA211

Commit message: Shunt_Cuk fixed _Switchs of the cuk fixed_ _Added isolation between the high voltage and the low voltage_
Parts:
- removed C12: 100nF, MCCplaca Shunt:C_0805_2012Metric_Pad1.29x1.40mm_HandSolder, symbol Device:C_Small
- removed R106, R108: 0R, Jumper:SolderJumper-2_P1.3mm_Open_Pad1.0x1.5mm, symbol Device:R_Small
- removed U6: INA211, MCCplaca Shunt:INA211BIDCKR, symbol Mcc18-rescue:INA211_DCK_6-INA211BIDCKR-Mcc18-rescue
- added C? (x2): 100nF, MCC:C_0805_2012Metric_Pad1.29x1.40mm_HandSolder, symbol Device:C_Small
- added L?: L_Small, Inductor_SMD:L_0805_2012Metric_Pad1.29x1.40mm_HandSolder, symbol Device:L_Small
- U1: symbol Mcc18-rescue:INA240-ina240_soic8-Mcc18-rescue -> Mcc18-rescue:INA240-ina240_soic8-Mcc18-rescue-Mcc18-rescue
Connections:
- net labels removed: INA211_OUT
- wire segments 254 -> 252

Commit message: Fixed errors
Parts:
- U1: symbol Mcc18-rescue:INA240-ina240_soic8-Mcc18-rescue-Mcc18-rescue -> Mcc18-rescue:INA240-ina240_soic8-Mcc18-rescue-Mcc18-rescue-Mcc18-rescue
Connections:
- wire segments 252 -> 253
Changed lines of the file:
@@
 Current Sensor\n
 $Comp
-L Mcc18-rescue:INA240-ina240_soic8-Mcc18-rescue-Mcc18-rescue U1
+L Mcc18-rescue:INA240-ina240_soic8-Mcc18-rescue-Mcc18-rescue-Mcc18-rescue U1
 U 1 1 5B114902
 P 7725 5700
@@
 Text Label 8325 6050 0    39   ~ 0
 INA240_OUT
-$Comp
-L power:+5VA #PWR0117
-U 1 1 5B575A82
-P 8400 5525
-F 0 "#PWR0117" H 8400 5375 50  0001 C CNN
-F 1 "+5VA" H 8415 5698 50  0000 C CNN
-F 2 "" H 8400 5525 50  0001 C CNN
-F 3 "" H 8400 5525 50  0001 C CNN
-	1    8400 5525
-	1    0    0    -1
-$EndComp
 $Comp
 L Device:R_Small R105
@@
 Wire Wire Line
 	8400 5525 8400 5950
-Connection ~ 8400 5525
 Wire Wire Line
 	3225 6850 3350 6850
@@
 	10400 5600 10550 5600
 $Comp
-L power:+5VA #PWR?
-U 1 1 5B29367F
-P 9700 5475
-F 0 "#PWR?" H 9700 5325 50  0001 C CNN
-F 1 "+5VA" H 9715 5603 50  0000 L CNN
-F 2 "" H 9700 5475 50  0001 C CNN
-F 3 "" H 9700 5475 50  0001 C CNN
-	1    9700 5475
-	1    0    0    -1
-$EndComp
-$Comp
 L power:+5V #PWR?
 U 1 1 5B293685
@@
 $EndComp
 Wire Wire Line
-	9700 5475 9700 5600
-Wire Wire Line
-	9700 5600 9800 5600
+	8800 5600 8800 5525
+Wire Wire Line
+	8800 5525 8550 5525
+Wire Wire Line
+	8800 5600 9800 5600
+Connection ~ 8550 5525
 $EndSCHEMATC

Commit message: finalized shunt cuk
Parts:
- gave numbers to parts that had none: 3
Changed lines of the file:
@@
 	8750 5050 8950 5050
 $Comp
-L Device:C_Small C?
+L Device:C_Small C13
 U 1 1 5B293655
 P 9800 5800
-F 0 "C?" H 9900 5825 39  0000 L CNN
+F 0 "C13" H 9900 5825 39  0000 L CNN
 F 1 "100nF" H 9900 5775 39  0000 L CNN
 F 2 "MCC:C_0805_2012Metric_Pad1.29x1.40mm_HandSolder" H 9800 5800 50  0001 C CNN
@@
 	10200 5600 10400 5600
 $Comp
-L power:GNDA #PWR?
+L power:GNDA #PWR0117
 U 1 1 5B293664
 P 9800 6000
-F 0 "#PWR?" H 9800 5750 39  0001 C CNN
+F 0 "#PWR0117" H 9800 5750 39  0001 C CNN
 F 1 "GNDA" H 9900 5825 50  0000 R CNN
 F 2 "" H 9800 6000 50  0001 C CNN
@@
 $EndComp
 $Comp
-L power:GND #PWR?
+L power:GND #PWR0118
 U 1 1 5B29366A
 P 10200 6000
-F 0 "#PWR?" H 10200 5750 50  0001 C CNN
+F 0 "#PWR0118" H 10200 5750 50  0001 C CNN
 F 1 "GND" H 10205 5827 50  0000 C CNN
 F 2 "" H 10200 6000 50  0001 C CNN
@@
 $EndComp
 $Comp
-L Device:L_Small L?
+L Device:L_Small L4
 U 1 1 5B293670
 P 10000 5600
-F 0 "L?" V 10100 5600 39  0000 C CNN
+F 0 "L4" V 10100 5600 39  0000 C CNN
 F 1 "L_Small" V 10050 5600 39  0000 C CNN
 F 2 "Inductor_SMD:L_0805_2012Metric_Pad1.29x1.40mm_HandSolder" H 10000 5600 50  0001 C CNN
@@
 $EndComp
 $Comp
-L Device:C_Small C?
+L Device:C_Small C12
 U 1 1 5B293676
 P 10200 5800
-F 0 "C?" H 10300 5825 39  0000 L CNN
+F 0 "C12" H 10300 5825 39  0000 L CNN
 F 1 "100nF" H 10300 5775 39  0000 L CNN
 F 2 "MCC:C_0805_2012Metric_Pad1.29x1.40mm_HandSolder" H 10200 5800 50  0001 C CNN
@@
 	10400 5600 10550 5600
 $Comp
-L power:+5V #PWR?
+L power:+5V #PWR0119
 U 1 1 5B293685
 P 10400 5500
-F 0 "#PWR?" H 10400 5350 50  0001 C CNN
+F 0 "#PWR0119" H 10400 5350 50  0001 C CNN
 F 1 "+5V" H 10415 5673 50  0000 C CNN
 F 2 "" H 10400 5500 50  0001 C CNN
