File: Hardware/Shunt_sensor/Cuk_converter/KiCad/Mcc18.sch (KiCad schematic (older format))
At the start: 94 parts, among them Q1 IRFP4321PbF, U1 INA240, U2 DRIVER_(INEP), U3 LM7812_TO220, U4 Signals_MCC, U5 ZCS

Commit message: Finlized signals basic routing
Parts:
- removed C6, C7: 100nF, Capacitor_SMD:C_0805_2012Metric_Pad1.15x1.40mm_HandSolder, symbol Device:C_Small
- removed L2: L_Small, Inductor_SMD:L_0805_2012Metric_Pad1.15x1.40mm_HandSolder, symbol Device:L_Small
- removed R107, R111: 0R, Jumper:SolderJumper-2_P1.3mm_Open_Pad1.0x1.5mm, symbol Device:R_Small
- removed R109: ??, Jumper:SolderJumper-2_P1.3mm_Bridged2Bar_Pad1.0x1.5mm, symbol Device:R_Small
- added JP4: VBat-Sen, Jumper:SolderJumper-2_P1.3mm_Open_Pad1.0x1.5mm, symbol Device:Jumper_NC_Small
- C1: value 100nF -> 1uF
- R110: value ?? -> 100
- Rshunt1: value 500uR -> 1500uR
- U3: footprint Package_TO_SOT_THT:TO-220-3_Horizontal_TabDown -> MCCplaca:TO-220-3_Horizontal_TabDown_SMD
Connections:
- wire segments 302 -> 287

Commit message: Added fill zones
Parts:
- U4: footprint MCCplaca:Signals -> MCCplaca:SignalsBarrapinos_SMD; symbol MCC18:Signals_MCC-MCC18-Mcc18-rescue-Mcc18-rescue-Mcc18-rescue-Mcc18-rescue -> Signals:Signals
- U5: symbol MCC18:ZCS-ZCS-Mcc18-rescue -> Mcc18-rescue:ZCS-ZCS-Mcc18-rescue-MCC18
Changed lines of the file:
@@
 	2350 5250 2350 5200
 $Comp
-L MCC18:Signals_MCC-MCC18-Mcc18-rescue-Mcc18-rescue-Mcc18-rescue-Mcc18-rescue U4
+L Signals:Signals U4
 U 1 1 5B191CBF
 P 4375 5250
 F 0 "U4" H 4194 5365 50  0000 C CNN
 F 1 "Signals_MCC" H 4194 5274 50  0000 C CNN
-F 2 "MCCplaca:Signals" H 4375 5250 50  0001 C CNN
+F 2 "MCCplaca:SignalsBarrapinos_SMD" H 4375 5250 50  0001 C CNN
 F 3 "" H 4375 5250 50  0001 C CNN
 	1    4375 5250
@@
 	1750 6800 1800 6800
 $Comp
-L MCC18:ZCS-ZCS-Mcc18-rescue U5
+L Mcc18-rescue:ZCS-ZCS-Mcc18-rescue-MCC18 U5
 U 1 1 5B16184F
 P 1300 5000

Commit message: Finalized first version PCB
Parts:
- removed JP2: MosfetOn, Jumper:SolderJumper-2_P1.3mm_Open_TrianglePad1.0x1.5mm, symbol Device:Jumper_NC_Small
- removed JP3: Diode On, Jumper:SolderJumper-2_P1.3mm_Open_Pad1.0x1.5mm, symbol Device:Jumper_NC_Small
- removed Rg2: 10k, Resistor_SMD:R_0805_2012Metric_Pad1.15x1.40mm_HandSolder, symbol Device:R_Small
- added JP5: ON/OFF, TerminalBlock:TerminalBlock_bornier-2_P5.08mm, symbol Device:Jumper_NC_Small
- added TP13, TP14: TP, TestPoint:TestPoint_Pad_2.0x2.0mm, symbol Connector:TestPoint_Probe
- C1: footprint Capacitor_SMD:C_0805_2012Metric_Pad1.15x1.40mm_HandSolder -> Capacitor_SMD:C_2512_6332Metric_Pad1.52x3.35mm_HandSolder
- D1: footprint MCCplaca:TO-247-3_Horizontal_TabUp -> Package_TO_SOT_THT:TO-247-3_Horizontal_TabUp
- JP1: value Diode On -> VBat-Sen
- L1, L3: footprint Inductor_SMD:L_0805_2012Metric_Pad1.15x1.40mm_HandSolder -> Jumper:SolderJumper-2_P1.3mm_Open_Pad1.0x1.5mm
- Rshunt1: footprint MCCplaca Shunt:PML100HZPJV0L5 -> MCCplaca:PML100HZPJV0L5
- TP1, TP10, TP11, TP12, TP2, TP3, TP4, TP5, TP6, TP7, TP8, TP9: value TestPoint_Probe -> TP; footprint TestPoint:TestPoint_Pad_D1.0mm -> TestPoint:TestPoint_Pad_2.0x2.0mm
- U1: symbol INA240:INA240-ina240_soic8-Mcc18-rescue-Mcc18-rescue-Mcc18-rescue -> Mcc18-rescue:INA240-ina240_soic8-Mcc18-rescue-Mcc18-rescue-Mcc18-rescue-Mcc18-rescue
- U2: footprint MCCplaca:Driver_(INEP)_SMD -> MCCplaca:Driver_(INEP)
- U3: footprint MCCplaca:TO-220-3_Horizontal_TabDown_SMD -> MCCplaca:TO-220-3_Horizontal_TabDown
- U4: footprint MCCplaca:SignalsBarrapinos_SMD -> MCCplaca:SignalsBarrapinosGrande; symbol Signals:Signals -> MCC18:Signals_MCC-MCC18-Mcc18-rescue-Mcc18-rescue-Mcc18-rescue-Mcc18-rescue
- U5: footprint MCCplaca:ZCS18 -> MCCplaca:ZCS18_Handsoldering; symbol Mcc18-rescue:ZCS-ZCS-Mcc18-rescue-MCC18 -> MCC18:ZCS-ZCS-Mcc18-rescue
Connections:
- net labels added: Gate, Source
- net labels removed: HG, HS, LG
- wire segments 287 -> 283
- no-connect marks 22 -> 21

Commit message: final adjusted for cnc.
Connections:
- wire segments 283 -> 284
Changed lines of the file:
@@
 Wire Wire Line
 	10175 3825 10400 3825
+$Comp
+L power:GNDA #PWR0126
+U 1 1 5B8A1A3D
+P 3600 7450
+F 0 "#PWR0126" H 3600 7200 39  0001 C CNN
+F 1 "GNDA" H 3605 7277 50  0000 C CNN
+F 2 "" H 3600 7450 50  0001 C CNN
+F 3 "" H 3600 7450 50  0001 C CNN
+	1    3600 7450
+	1    0    0    -1
+$EndComp
+$Comp
+L power:GND #PWR0127
+U 1 1 5B8A23AB
+P 3850 7450
+F 0 "#PWR0127" H 3850 7200 50  0001 C CNN
+F 1 "GND" H 3855 7277 50  0000 C CNN
+F 2 "" H 3850 7450 50  0001 C CNN
+F 3 "" H 3850 7450 50  0001 C CNN
+	1    3850 7450
+	1    0    0    -1
+$EndComp
+Wire Wire Line
+	3600 7450 3850 7450
 $EndSCHEMATC

Commit message: Fixed signals tracks
Parts:
- U1: symbol Mcc18-rescue:INA240-ina240_soic8-Mcc18-rescue-Mcc18-rescue-Mcc18-rescue-Mcc18-rescue -> Mcc18-rescue:INA240-ina240_soic8-Mcc18-rescue-Mcc18-rescue-Mcc18-rescue-Mcc18-rescue-Mcc18-rescue
Changed lines of the file:
@@
 Current Sensor\n
 $Comp
-L Mcc18-rescue:INA240-ina240_soic8-Mcc18-rescue-Mcc18-rescue-Mcc18-rescue-Mcc18-rescue U1
+L Mcc18-rescue:INA240-ina240_soic8-Mcc18-rescue-Mcc18-rescue-Mcc18-rescue-Mcc18-rescue-Mcc18-rescue U1
 U 1 1 5B114902
 P 7725 5700
